File: fg-11.kicad_pcb (KiCad board)
At the start: 2 copper layers, 321.3 x 128.9 mm, 75 parts, among them J1 Conn_02x05_Counter_Clockwise, J2 Conn_02x05_Counter_Clockwise, U1 ProMicro

Commit message: Correct order of right thumb switches and reroute tracks to simplify.
Parts:
- moved MX34 44.2 mm to (221.0, 65.4), turned to 45 degrees
- moved MX36 44.2 mm to (264.2, 55.9), turned to 0 degrees
- moved D36 33.2 mm to (273.1, 51.2)
- moved D34 21.5 mm to (230.5, 50.8)
- moved D18 11.5 mm to (163.8, 48.3)
- moved D17 10.9 mm to (158.1, 48.3)
- moved D35 10.2 mm to (253.4, 50.5)
- moved D16 4.02 mm to (138.4, 48.3)
Routing:
- net row4-j2: track 24.8 -> 69.2 mm, vias 0 -> 3
- net col8-j2: track 171.0 -> 137.5 mm, vias 1 -> 0
- net col4: track 207.8 -> 181.0 mm, vias 2 -> 1
- net col6-j2: track 88.8 -> 115.5 mm
- net col7-j2: track 150.7 -> 131.3 mm, vias 1 -> 0
- net Net-(D34-Pad2): track 33.2 -> 16.0 mm
- net Net-(D36-Pad2): track 27.2 -> 12.2 mm
- net col1: track 224.8 -> 211.1 mm, vias 0 -> 1
- net col10-j1: track 45.7 -> 33.2 mm
- net row4: track 76.4 -> 84.2 mm, vias 1 -> 0
- net col3: track 208.9 -> 201.2 mm
- net col9-j1: track 41.2 -> 35.2 mm
- net row2: track 157.8 -> 152.6 mm, vias 5 -> 6
- net col5: track 130.0 -> 134.8 mm
- net Net-(D35-Pad2): track 17.4 -> 12.8 mm
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
Commit message: Various improvements.
- Reduce the spacing between the keys.
- Flip the pro-micro footprint (to reveal reset buttons for elite-c etc.)
- Rework the tracks to simplify them.
- Redo the cuts to make them more consistent.
Parts:
- U1: moved to B.Cu
- moved MX34 23.9 mm to (232.3, 86.5)
- moved MX18 23.4 mm to (162.7, 86.5)
- moved D34 19.4 mm to (249.6, 47.0)
- moved MX35 17.2 mm to (245.7, 73.0), turned to 45 degrees
- moved MX17 17.1 mm to (149.2, 73.0), turned to 315 degrees
- moved D17 11.1 mm to (148.0, 43.8)
- moved D18 10.5 mm to (154.3, 43.8)
- moved D21 9.38 mm to (304.2, -23.5), turned to 0 degrees
- moved D26 8.84 mm to (304.2, -4.45), turned to 0 degrees
- moved D31 8.47 mm to (304.2, 14.6), turned to 0 degrees
- moved D20 8.28 mm to (285.1, -23.5), turned to 0 degrees
- moved D25 7.67 mm to (285.1, -4.45), turned to 0 degrees
- moved J2 7.65 mm to (243.8, 24.8)
- moved D4 7.65 mm to (113.0, -22.2), turned to 0 degrees
- moved D30 7.24 mm to (285.1, 14.6), turned to 0 degrees
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Routing:
- net col1: track 211.1 -> 138.9 mm
- net col2: track 181.5 -> 129.9 mm, vias 1 -> 2
- net Net-(D34-Pad2): track 16.0 -> 44.2 mm
- net Net-(D18-Pad2): track 28.9 -> 55.0 mm
- net row1: track 161.8 -> 136.6 mm
- net Net-(D17-Pad2): track 15.1 -> 37.7 mm
- net row3: track 149.2 -> 127.8 mm, vias 6 -> 5
- net row4-j2: track 69.2 -> 48.0 mm
- net col5: track 134.8 -> 153.5 mm, vias 0 -> 1
- net col7-j2: track 131.3 -> 150.0 mm
- net col3: track 201.2 -> 182.8 mm, vias 2 -> 1
- net col8-j2: track 137.5 -> 119.9 mm
- net col4: track 181.0 -> 163.7 mm
- net row4: track 84.2 -> 68.4 mm
- net col10-j2: track 148.5 -> 133.6 mm
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Other:
- board size 321.3 x 128.9 mm -> 311.1 x 149.5 mm

Commit message: Add mount holes, plate, and back.
Parts:
- added MX1: MX-NoLED, kbd:SW_Hole, F.Cu at (54.0, 136.5)
- added MX10: MX-NoLED, kbd:SW_Hole, F.Cu at (130.2, 155.6)
- added MX11: MX-NoLED, kbd:SW_Hole, F.Cu at (54.0, 174.6)
- added MX12: MX-NoLED, kbd:SW_Hole, F.Cu at (73.0, 174.6)
- added MX13: MX-NoLED, kbd:SW_Hole, F.Cu at (92.1, 155.6)
- added MX14: MX-NoLED, kbd:SW_Hole, F.Cu at (111.1, 155.6)
- added MX15: MX-NoLED, kbd:SW_Hole, F.Cu at (130.2, 174.6)
- added MX16: MX-NoLED, kbd:SW_Hole, F.Cu at (130.2, 203.2)
- added MX17: MX-NoLED, kbd:SW_Hole, F.Cu at (149.2, 225.4)
- added MX18: MX-NoLED, kbd:SW_Hole, F.Cu at (162.7, 238.9)
- added MX2: MX-NoLED, kbd:SW_Hole, F.Cu at (73.0, 136.5)
- added MX3: MX-NoLED, kbd:SW_Hole, F.Cu at (92.1, 117.5)
- added MX4: MX-NoLED, kbd:SW_Hole, F.Cu at (111.1, 117.5)
- added MX5: MX-NoLED, kbd:SW_Hole, F.Cu at (130.2, 136.5)
- added MX6: MX-NoLED, kbd:SW_Hole, F.Cu at (54.0, 155.6)
- added MX7: MX-NoLED, kbd:SW_Hole, F.Cu at (73.0, 155.6)
- added MX8: MX-NoLED, kbd:SW_Hole, F.Cu at (92.1, 136.5)
- added MX9: MX-NoLED, kbd:SW_Hole, F.Cu at (111.1, 136.5)
- added Ref**: Val**, kbd:M2_Hole_TH, F.Cu at (225.4, 123.8)
- added Ref**: Val**, kbd:M2_Hole_TH, F.Cu at (79.4, 123.8)
- added Ref**: Val**, kbd:spacer_m2, B.Cu at (331.5, 12.7)
- added Ref**: Val**, kbd:spacer_m2, B.Cu at (259.1, 36.2)
- added Ref**: Val**, kbd:spacer_m2, B.Cu at (271.1, -28.6)
- added Ref**: Val**, kbd:spacer_m2, B.Cu at (315.6, -28.6)
- added Ref**: Val**, kbd:spacer_m2, B.Cu at (244.5, 85.1)
- added Ref**: Val**, kbd:spacer_m2, F.Cu at (150.5, 85.1)
- added Ref**: Val**, kbd:spacer_m2, F.Cu at (135.9, 36.2)
- added Ref**: Val**, kbd:spacer_m2, F.Cu at (63.5, 12.7)
- added Ref**: Val**, kbd:spacer_m2, F.Cu at (123.8, -28.6)
- added Ref**: Val**, kbd:M2_Hole_TH, F.Cu at (296.5, 237.5)
- added Ref**: Val**, kbd:spacer_m2, F.Cu at (79.4, -28.6)
- added Ref**: Val**, kbd:M2_Hole_TH, F.Cu at (209.6, 165.1)
- added Ref**: Val**, kbd:M2_Hole_TH, F.Cu at (269.9, 123.8)
- added Ref**: Val**, kbd:M2_Hole_TH, F.Cu at (281.9, 188.6)
- added Ref**: Val**, kbd:M2_Hole_TH, F.Cu at (63.5, 165.1)
- added Ref**: Val**, kbd:M2_Hole_TH, F.Cu at (135.9, 188.6)
- added Ref**: Val**, kbd:M2_Hole_TH, F.Cu at (150.5, 237.5)
- added Ref**: Val**, kbd:M2_Hole_TH, F.Cu at (123.8, 123.8)
- moved J1 2.54 mm to (152.4, 24.1)
- moved U1 2.54 mm to (153.7, -8.89)
- moved D32 1.27 mm to (330.2, 19.7)
- moved D33 1.27 mm to (349.2, 19.7)
Routing:
- net row3: track 127.8 -> 132.9 mm
- net col1: track 138.9 -> 142.4 mm
- net col5: track 153.5 -> 156.2 mm
- net col4: track 163.7 -> 166.2 mm
- net row2: track 156.1 -> 158.6 mm
- net col2: track 129.9 -> 132.1 mm
- net Net-(D33-Pad2): track 11.8 -> 9.75 mm
- net Net-(D32-Pad2): track 12.6 -> 11.3 mm
- net col10-j2: track 133.6 -> 134.7 mm
- net row1: track 136.6 -> 137.6 mm
- net col3: track 182.8 -> 183.9 mm
- net col6-j2: track 129.0 -> 128.2 mm
- net col9-j2: track 115.3 -> 116.0 mm
- net col7-j2: track 150.0 -> 150.5 mm
- net row3-j2: track 118.9 -> 119.5 mm
Other:
- board size 311.1 x 149.5 mm -> 311.1 x 301.9 mm
- board text added: "FG-11 Rev01"

Commit message: Last commit with plates.
Parts:
- removed the MX1 at (54.0, 136.5)
- removed the MX10 at (130.2, 155.6)
- removed the MX11 at (54.0, 174.6)
- removed the MX12 at (73.0, 174.6)
- removed the MX13 at (92.1, 155.6)
- removed the MX14 at (111.1, 155.6)
- removed the MX15 at (130.2, 174.6)
- removed the MX16 at (130.2, 203.2)
- removed the MX17 at (149.2, 225.4)
- removed the MX18 at (162.7, 238.9)
- removed the MX2 at (73.0, 136.5)
- removed the MX3 at (92.1, 117.5)
- removed the MX4 at (111.1, 117.5)
- removed the MX5 at (130.2, 136.5)
- removed the MX6 at (54.0, 155.6)
- removed the MX7 at (73.0, 155.6)
- removed the MX8 at (92.1, 136.5)
- removed the MX9 at (111.1, 136.5)
- added mount1: , future-gadget-11:SW_Hole_Choc, F.Cu at (54.0, 136.5)
- added mount10: , future-gadget-11:SW_Hole_Choc, F.Cu at (130.2, 155.6)
- added mount11: , future-gadget-11:SW_Hole_Choc, F.Cu at (54.0, 174.6)
- added mount12: , future-gadget-11:SW_Hole_Choc, F.Cu at (73.0, 174.6)
- added mount13: , future-gadget-11:SW_Hole_Choc, F.Cu at (92.1, 155.6)
- added mount14: , future-gadget-11:SW_Hole_Choc, F.Cu at (111.1, 155.6)
- added mount15: , future-gadget-11:SW_Hole_Choc, F.Cu at (130.2, 174.6)
- added mount16: , future-gadget-11:SW_Hole_Choc, F.Cu at (130.2, 203.2)
- added mount17: , future-gadget-11:SW_Hole_Choc, F.Cu at (149.2, 225.4)
- added mount18: , future-gadget-11:SW_Hole_Choc, F.Cu at (162.7, 238.9)
- added mount2: , future-gadget-11:SW_Hole_Choc, F.Cu at (73.0, 136.5)
- added mount3: , future-gadget-11:SW_Hole_Choc, F.Cu at (92.1, 117.5)
- added mount4: , future-gadget-11:SW_Hole_Choc, F.Cu at (111.1, 117.5)
- added mount5: , future-gadget-11:SW_Hole_Choc, F.Cu at (130.2, 136.5)
- added mount6: , future-gadget-11:SW_Hole_Choc, F.Cu at (54.0, 155.6)
- added mount7: , future-gadget-11:SW_Hole_Choc, F.Cu at (73.0, 155.6)
- added mount8: , future-gadget-11:SW_Hole_Choc, F.Cu at (92.1, 136.5)
- added mount9: , future-gadget-11:SW_Hole_Choc, F.Cu at (111.1, 136.5)

Commit message: Panelize PCB and add SVG files for plates.
Parts:
- removed the MX31 at (302.9, 3.17)
- removed the Ref** at (225.4, 123.8)
- removed the Ref** at (79.4, 123.8)
- removed the Ref** at (331.5, 12.7)
- removed the Ref** at (259.1, 36.2)
- removed the Ref** at (271.1, -28.6)
- removed the Ref** at (315.6, -28.6)
- removed the Ref** at (244.5, 85.1)
- removed the Ref** at (296.5, 237.5)
- removed the Ref** at (209.6, 165.1)
- removed the Ref** at (269.9, 123.8)
- removed the Ref** at (281.9, 188.6)
- removed the Ref** at (63.5, 165.1)
- removed the Ref** at (135.9, 188.6)
- removed the Ref** at (150.5, 237.5)
- removed the Ref** at (123.8, 123.8)
- removed mount1, mount10, mount11, mount12, mount13, mount14, mount15, mount16, mount17, mount18, mount2, mount4, mount5, mount6, mount7, mount8, mount9: , future-gadget-11:SW_Hole_Choc
- added Ref**: Val**, kbd:spacer_m2, B.Cu at (-53.3, 24.1)
- added Ref**: Val**, kbd:spacer_m2, B.Cu at (19.1, 0.64)
- added Ref**: Val**, kbd:spacer_m2, B.Cu at (6.99, 65.4)
- added Ref**: Val**, kbd:spacer_m2, B.Cu at (-37.5, 65.4)
- added Ref**: Val**, kbd:spacer_m2, B.Cu at (33.7, -48.3)
- added mouse-bite-2mm-slot: VAL**, panelization:mouse-bite-2mm-slot, F.Cu at (41.2, -15.8)
- added mouse-bite-2mm-slot: VAL**, panelization:mouse-bite-2mm-slot, F.Cu at (41.3, 4.45)
- MX31: renamed from mount3; value (none) -> MX-NoLED; footprint future-gadget-11:SW_Hole_Choc -> kbd:ChocV1_V2_Hotswap
- moved D23 427.2 mm to (-71.1, 56.5), turned to 90 degrees
- moved D28 422.1 mm to (-71.1, 37.5), turned to 90 degrees
- moved D33 420.4 mm to (-71.1, 17.1), turned to 90 degrees
- moved MX23 409.6 mm to (-62.9, 52.7), turned to 180 degrees
- moved MX28 405.0 mm to (-62.9, 33.7), turned to 180 degrees
- moved MX33 403.9 mm to (-62.9, 14.6), turned to 180 degrees
- moved D22 389.8 mm to (-52.1, 56.5), turned to 90 degrees
- moved D27 384.2 mm to (-52.1, 37.5), turned to 90 degrees
- moved D32 382.3 mm to (-52.1, 17.1), turned to 90 degrees
- moved MX22 372.1 mm to (-43.8, 52.7), turned to 180 degrees
- moved MX27 367.0 mm to (-43.8, 33.7), turned to 180 degrees
- moved MX32 365.8 mm to (-43.8, 14.6), turned to 180 degrees
- moved MX21 344.6 mm to (-24.8, 71.8), turned to 180 degrees
- moved D21 340.7 mm to (-26.0, 60.3), turned to 180 degrees
- moved MX26 334.8 mm to (-24.8, 52.7), turned to 180 degrees
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Other:
- board size 311.1 x 301.9 mm -> 253.6 x 168.2 mm

Commit message: First go at revision 2.
Revision 2 has several goals:

- Shift the index and ring finger one column outward, giving the
  index finger two columns each and the little fingers one each.
- Flip the controller. It was handy to have it the other way up for
  access to the reset button on an elite-c, but the on-board LED
  is bright blue and distracting.
- Add a reset button. By doing this any pro-micro footprint
  controller can now be used.
- Re-align the diodes. Many weren't quite aligned in rev-1 and it
  irked me.
Parts:
- removed the Ref** at (-53.3, 24.1)
- removed the Ref** at (19.1, 0.64)
- removed the Ref** at (6.99, 65.4)
- removed the Ref** at (-37.5, 65.4)
- removed the Ref** at (33.7, -48.3)
- removed the Ref** at (150.5, 85.1)
- removed the Ref** at (135.9, 36.2)
- added Ref**: Val**, kbd:spacer_m2, B.Cu at (-36.2, 36.2)
- added Ref**: Val**, kbd:spacer_m2, B.Cu at (12.7, 19.1)
- added Ref**: Val**, kbd:spacer_m2, B.Cu at (-25.4, -31.8)
- added Ref**: Val**, kbd:spacer_m2, B.Cu at (25.4, -31.8)
- added Ref**: Val**, kbd:spacer_m2, B.Cu at (-48.9, 85.1)
- added Ref**: Val**, kbd:spacer_m2, F.Cu at (131.4, 85.1)
- added Ref**: Val**, kbd:spacer_m2, F.Cu at (69.8, 19.1)
- added reset1: SW_Push, kbd:ResetSW_1side, F.Cu at (137.8, 59.7)
- U1: moved to F.Cu
- moved MX34 173.1 mm to (-61.1, 86.5), turned to 45 degrees
- moved MX35 135.4 mm to (-47.6, 73.0), turned to 45 degrees
- moved D23 128.8 mm to (31.8, -21.0), turned to 270 degrees
- moved MX23 114.3 mm to (28.6, -15.9), turned to 0 degrees
- moved D28 110.1 mm to (31.8, -1.91), turned to 270 degrees
- moved MX21 107.8 mm to (-9.53, -34.9), turned to 0 degrees
- moved D33 102.9 mm to (31.8, 17.1), turned to 270 degrees
- moved D22 102.6 mm to (11.4, -24.1), turned to 0 degrees
- moved MX22 102.6 mm to (9.53, -34.9), turned to 0 degrees
- moved D34 101.1 mm to (-46.4, 57.8), turned to 270 degrees
- moved D35 96.5 mm to (-43.2, 57.8), turned to 270 degrees
- moved MX28 96.4 mm to (28.6, 3.17), turned to 0 degrees
- moved D19 92.2 mm to (-44.5, -21.0), turned to 270 degrees
- moved J2 92.0 mm to (-53.3, 40.0), turned to 0 degrees
- moved MX19 91.8 mm to (-47.6, -15.9), turned to 0 degrees
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Connections:
- U1 pad 18: col5 -> row4
- U1 pad 5: row1 -> row3
- U1 pad 7: row3 -> col5
- U1 pad 8: row4 -> row1
Routing:
- net Net-(U1-Pad23): track 0.00 -> 110.4 mm
- net Net-(U1-Pad22): track 0.00 -> 106.3 mm
- net col8-j1: track 34.9 -> 125.8 mm
- net col6-j1: track 37.4 -> 127.7 mm
- net col10-j1: track 32.3 -> 117.4 mm
- net col7-j1: track 39.5 -> 123.4 mm
- net col9-j1: track 40.5 -> 120.2 mm
- net row4: track 68.4 -> 140.2 mm
- net col3: track 183.9 -> 123.3 mm
- net col4: track 166.2 -> 113.3 mm, vias 1 -> 0
- net col2: track 132.1 -> 84.6 mm, vias 2 -> 1
- net col7-j2: track 150.5 -> 104.3 mm
- net col5: track 156.2 -> 120.5 mm, vias 1 -> 0
- net col1: track 142.4 -> 108.0 mm
- net row3: track 132.9 -> 167.1 mm
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Other:
- board size 253.6 x 168.2 mm -> 236.8 x 149.5 mm
